Commit message: cleaned code

File: urdf/turtlebot3_burger.gazebo.xacro (robot description, xacro)
@@ -42,47 +42,4 @@
     </sensor>
     <material>Gazebo/FlatBlack</material>
-  </gazebo>
-  <gazebo reference="kinect_link">
-    <sensor type="depth" name="kinect">
-      <always_on>true</always_on>
-      <visualize>true</visualize>
-      <camera>
-        <horizontal_fov>1.047</horizontal_fov>
-        <image>
-          <width>640</width>
-          <height>480</height>
-          <format>R8G8B8</format>
-        </image>
-        <depth_camera>
-        </depth_camera>
-        <clip>
-          <near>0.1</near>
-          <far>100</far>
-        </clip>
-      </camera>
-      <plugin name="kinect_plugin" filename="libgazebo_ros_openni_kinect.so">
-        <baseline>0.2</baseline>
-        <alwaysOn>true</alwaysOn>
-        <updateRate>10.0</updateRate>
-        <cameraName>kinect</cameraName>
-        <frameName>kinect_link</frameName>
-        <imageTopicName>rgb/image_raw</imageTopicName>
-        <depthImageTopicName>depth/image_raw</depthImageTopicName>
-        <pointCloudTopicName>depth/points</pointCloudTopicName>
-        <cameraInfoTopicName>rgb/camera_info</cameraInfoTopicName>
-        <depthImageCameraInfoTopicName>depth/camera_info</depthImageCameraInfoTopicName>
-        <pointCloudCutoff>0.4</pointCloudCutoff>
-              <hackBaseline>0.07</hackBaseline>
-              <distortionK1>0.0</distortionK1>
-              <distortionK2>0.0</distortionK2>
-              <distortionK3>0.0</distortionK3>
-              <distortionT1>0.0</distortionT1>
-              <distortionT2>0.0</distortionT2>
-          <CxPrime>0.0</CxPrime>
-          <Cx>0.0</Cx>
-          <Cy>0.0</Cy>
-          <focalLength>0.0</focalLength>
-      </plugin>
-      </sensor>
   </gazebo>
   <gazebo>

File: urdf/turtlebot3_burger.urdf.xacro (robot description, xacro)
@@ -140,5 +140,5 @@
     </inertial>
   </link>
-  <joint name="kinect_joint" type="fixed">
+  <!--joint name="kinect_joint" type="fixed">
     <parent link="base_link"/>
     <child link="kinect_link"/>
@@ -166,4 +166,4 @@
                izz="0.001" />
     </inertial>
-  </link>
+  </link-->
 </robot>
